Commit message: wip transform manager

File: src/vehicle_launch/donkeysim_launch/param/donkeycar.urdf (robot description, URDF)
Before this commit: robot donkeycar, 6 links, 5 joints
Links:
- removed link map
Joints:
- removed joint map_joint
- joint base_footprint_joint: origin xyz=0 0 0 rpy=0 0 0 -> xyz=0 0 -0.5 rpy=0 0 0
